File: schemes/scheme to print.brd (EAGLE design)
At the start: 72 parts

Commit message: pull-up resistors
Parts:
- added C7, C8: 100n, rcl:C0805
- added IC7, IC8: (no value), HC-05:HC-05
- added KEY_OUT6, KEY_OUT7, RESET6, RESET7: M01PTH_LONGPAD, SparkFun:1X01_LONGPAD
- added KEY_ZWORKA6, KEY_ZWORKA7, RX/TX6, RX/TX7, SUPPLY6, SUPPLY7: (no value), SparkFun:1X02_LONGPADS
- added LED13, LED15: RED, led:CHIPLED_0805
- added LED14, LED16: GREEN, led:CHIPLED_0805
- added R13, R14, R17, R18, R21, R22, R25, R26, R29, R30: 470, rcl:R0805
- added R15, R16, R19, R20, R23, R24, R27, R28, R31, R32: 10k, rcl:R0805
- added U$7, U$8: (no value), synergia_logo:SYNERGIA_12MM
- R11, R12, R3, R4, R7, R8: value 470 -> 10k
- moved R5 74.7 mm to (71.1, 52.1)
- moved R6 74.7 mm to (67.3, 52.1)
- moved R11 72.8 mm to (34.3, 16.5), turned to 0 degrees
- moved R8 69.9 mm to (95.2, 66.0), turned to 0 degrees
- moved R12 68.9 mm to (39.4, 16.5), turned to 0 degrees
- moved R7 66.7 mm to (90.2, 66.0), turned to 0 degrees
- moved R10 49.5 mm to (11.4, 2.54)
- moved R9 49.5 mm to (15.2, 2.54)
- moved R3 38.2 mm to (34.3, 66.0), turned to 0 degrees
- moved R4 30.1 mm to (39.4, 66.0), turned to 0 degrees
- moved KEY_OUT1 1.27 mm to (97.8, 57.1)
- moved KEY_OUT3 1.27 mm to (97.8, 7.62)
- moved KEY_ZWORKA1 1.27 mm to (97.8, 50.8)
- moved KEY_ZWORKA3 1.27 mm to (97.8, 1.27)
- moved LED4 1.27 mm to (71.1, 47.0)
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Connections:
- new net 3.3V6: C7.1, IC7.3V3, KEY_ZWORKA6.1, R27.2, R28.2, SUPPLY6.1
- new net 3.3V7: C8.1, IC8.3V3, KEY_ZWORKA7.1, R31.2, R32.2, SUPPLY7.1
- new net GND6: C7.2, IC7.GND@1, IC7.GND@2, IC7.GND@3, LED13.C, LED14.C, SUPPLY6.2
- new net GND7: C8.2, IC8.GND@1, IC8.GND@2, IC8.GND@3, LED15.C, LED16.C, SUPPLY7.2
- new net N$49: IC7.PIO11(KEY), KEY_OUT6.1, KEY_ZWORKA6.2
- new net N$50: IC7.PIO8(LED1), R25.1
- new net N$51: IC7.PIO9(LED2), R26.1
- new net N$52: LED13.A, R26.2
- new net N$53: LED14.A, R25.2
- new net N$54: IC7.TX, R27.1, RX/TX6.2
- new net N$55: IC7.RX, R28.1, RX/TX6.1
- new net N$56: IC7.RESET, RESET6.1
- new net N$57: IC8.PIO11(KEY), KEY_OUT7.1, KEY_ZWORKA7.2
- new net N$58: IC8.PIO8(LED1), R29.1
- new net N$59: IC8.PIO9(LED2), R30.1
- new net N$60: LED15.A, R30.2
- new net N$61: LED16.A, R29.2
- new net N$62: IC8.TX, R31.1, RX/TX7.2
- new net N$63: IC8.RX, R32.1, RX/TX7.1
- new net N$64: IC8.RESET, RESET7.1
- net 3.3V: now also R3.2, R4.2
- net 3.3V1: now also R7.2, R8.2
- net 3.3V2: now also R11.2, R12.2
- net 3.3V3: now also R15.2, R16.2
- net 3.3V4: now also R19.2, R20.2
- net 3.3V5: now also R23.2, R24.2
- net N$10: now also R5.1; no longer R3.1
- net N$11: now also R6.1; no longer R4.1
- net N$12: now also R6.2; no longer R4.2
- net N$13: now also R5.2; no longer R3.2
- net N$14: now also R7.1
- net N$15: now also R8.1
- net N$18: now also R9.1; no longer R5.1
- net N$19: now also R10.1; no longer R6.1
- net N$20: now also R10.2; no longer R6.2
- net N$21: now also R9.2; no longer R5.2
- net N$22: now also R11.1
- net N$23: now also R12.1
- net N$26: now also R13.1; no longer R7.1
- net N$27: now also R14.1; no longer R8.1
- net N$28: now also R14.2; no longer R8.2
- net N$29: now also R13.2; no longer R7.2
- net N$30: now also R15.1
- net N$31: now also R16.1
- net N$34: now also R17.1; no longer R9.1
- net N$35: now also R18.1; no longer R10.1
- net N$36: now also R18.2; no longer R10.2
- net N$37: now also R17.2; no longer R9.2
- net N$38: now also R19.1
- net N$39: now also R20.1
- net N$42: now also R21.1; no longer R11.1
- net N$43: now also R22.1; no longer R12.1
- net N$44: now also R22.2; no longer R12.2
- net N$45: now also R21.2; no longer R11.2
- net N$46: now also R23.1
- net N$47: now also R24.1
- net N$7: now also R3.1
- net N$8: now also R4.1
Routing:
- net 3.3V6: track 0.00 -> 105.9 mm
- net 3.3V7: track 0.00 -> 105.9 mm
- net N$57: track 0.00 -> 66.8 mm
- net N$49: track 0.00 -> 66.8 mm
- net 3.3V2: track 42.6 -> 105.9 mm
- net 3.3V4: track 42.6 -> 105.9 mm
- net 3.3V5: track 42.6 -> 105.9 mm
- net 3.3V: track 42.6 -> 105.9 mm
- net 3.3V3: track 42.6 -> 105.9 mm
- net 3.3V1: track 42.6 -> 105.9 mm
- net N$55: track 0.00 -> 24.1 mm
- net N$63: track 0.00 -> 24.1 mm
- net N$54: track 0.00 -> 16.3 mm
- net N$62: track 0.00 -> 16.3 mm
- net N$8: track 11.3 -> 24.1 mm
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- added copper zone on layer 16, net GND6
- added copper zone on layer 16, net GND7
