File: schemes/scheme.brd (EAGLE design)
At the start: 100 x 80 mm, 12 parts

Commit message: pull-up resistors
Parts:
- added R3, R4: 10k, rcl:R0805
Connections:
- net 3.3V: now also R3.2, R4.2
- net N$7: now also R3.1
- net N$8: now also R4.1
Routing:
- net 3.3V: track 42.6 -> 105.9 mm
- net N$8: track 11.3 -> 24.1 mm
- net N$1: track 55.3 -> 66.8 mm
- net N$7: track 11.8 -> 16.3 mm
Changed lines of the file:
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@@
 <setting verticaltext="up"/>
 </settings>
-<grid distance="0.05" unitdist="inch" unit="inch" style="lines" multiple="1" display="no" altdistance="0.025" altunitdist="inch" altunit="inch"/>
+<grid distance="0.01" unitdist="inch" unit="inch" style="lines" multiple="1" display="no" altdistance="0.025" altunitdist="inch" altunit="inch"/>
 <layers>
 <layer number="1" name="Top" color="4" fill="1" visible="yes" active="yes"/>
@@
 <layer number="27" name="tValues" color="7" fill="1" visible="yes" active="yes"/>
 <layer number="28" name="bValues" color="7" fill="1" visible="yes" active="yes"/>
-<layer number="29" name="tStop" color="7" fill="3" visible="no" active="yes"/>
-<layer number="30" name="bStop" color="7" fill="6" visible="no" active="yes"/>
-<layer number="31" name="tCream" color="7" fill="4" visible="no" active="yes"/>
-<layer number="32" name="bCream" color="7" fill="5" visible="no" active="yes"/>
-<layer number="33" name="tFinish" color="6" fill="3" visible="no" active="yes"/>
-<layer number="34" name="bFinish" color="6" fill="6" visible="no" active="yes"/>
-<layer number="35" name="tGlue" color="7" fill="4" visible="no" active="yes"/>
-<layer number="36" name="bGlue" color="7" fill="5" visible="no" active="yes"/>
-<layer number="37" name="tTest" color="7" fill="1" visible="no" active="yes"/>
-<layer number="38" name="bTest" color="7" fill="1" visible="no" active="yes"/>
+<layer number="29" name="tStop" color="7" fill="3" visible="yes" active="yes"/>
+<layer number="30" name="bStop" color="7" fill="6" visible="yes" active="yes"/>
+<layer number="31" name="tCream" color="7" fill="4" visible="yes" active="yes"/>
+<layer number="32" name="bCream" color="7" fill="5" visible="yes" active="yes"/>
+<layer number="33" name="tFinish" color="6" fill="3" visible="yes" active="yes"/>
+<layer number="34" name="bFinish" color="6" fill="6" visible="yes" active="yes"/>
+<layer number="35" name="tGlue" color="7" fill="4" visible="yes" active="yes"/>
+<layer number="36" name="bGlue" color="7" fill="5" visible="yes" active="yes"/>
+<layer number="37" name="tTest" color="7" fill="1" visible="yes" active="yes"/>
+<layer number="38" name="bTest" color="7" fill="1" visible="yes" active="yes"/>
 <layer number="39" name="tKeepout" color="4" fill="11" visible="yes" active="yes"/>
 <layer number="40" name="bKeepout" color="1" fill="11" visible="yes" active="yes"/>
@@
 <layer number="42" name="bRestrict" color="1" fill="10" visible="yes" active="yes"/>
 <layer number="43" name="vRestrict" color="2" fill="10" visible="yes" active="yes"/>
-<layer number="44" name="Drills" color="7" fill="1" visible="no" active="yes"/>
-<layer number="45" name="Holes" color="7" fill="1" visible="no" active="yes"/>
-<layer number="46" name="Milling" color="3" fill="1" visible="no" active="yes"/>
-<layer number="47" name="Measures" color="7" fill="1" visible="no" active="yes"/>
+<layer number="44" name="Drills" color="7" fill="1" visible="yes" active="yes"/>
+<layer number="45" name="Holes" color="7" fill="1" visible="yes" active="yes"/>
+<layer number="46" name="Milling" color="3" fill="1" visible="yes" active="yes"/>
+<layer number="47" name="Measures" color="7" fill="1" visible="yes" active="yes"/>
 <layer number="48" name="Document" color="7" fill="1" visible="yes" active="yes"/>
 <layer number="49" name="Reference" color="7" fill="1" visible="yes" active="yes"/>
@@
 <element name="SUPPLY" library="SparkFun" package="1X02_LONGPADS" value="" x="41.91" y="43.18" rot="R270"/>
 <element name="U$1" library="synergia_logo" package="SYNERGIA_12MM" value="" x="6.35" y="66.04" rot="MR270"/>
+<element name="R3" library="rcl" package="R0805" value="10k" x="34.29" y="66.04" rot="MR0"/>
+<element name="R4" library="rcl" package="R0805" value="10k" x="39.37" y="66.04" rot="MR0"/>
 </elements>
 <signals>
@@
 <contactref element="KEY_OUT" pad="1"/>
 <wire x1="41.91" y1="57.15" x2="41.91" y2="53.34" width="0.6096" layer="16"/>
-<wire x1="41.91" y1="57.15" x2="43.18" y2="58.42" width="0.6096" layer="16"/>
-<wire x1="43.18" y1="58.42" x2="44.45" y2="58.42" width="0.6096" layer="16"/>
-<wire x1="44.45" y1="58.42" x2="45.72" y2="59.69" width="0.6096" layer="16"/>
-<wire x1="45.72" y1="59.69" x2="45.72" y2="66.04" width="0.6096" layer="16"/>
-<wire x1="45.72" y1="66.04" x2="43.18" y2="68.58" width="0.6096" layer="16"/>
-<wire x1="43.18" y1="68.58" x2="17.78" y2="68.58" width="0.6096" layer="16"/>
-<wire x1="17.78" y1="68.58" x2="16.51" y2="67.31" width="0.6096" layer="16"/>
 <wire x1="16.51" y1="67.31" x2="16.51" y2="60.96" width="0.6096" layer="16"/>
 <wire x1="16.51" y1="60.96" x2="17.78" y2="59.69" width="0.6096" layer="16"/>
 <wire x1="17.78" y1="59.69" x2="18.93" y2="59.69" width="0.6096" layer="16"/>
 <wire x1="18.93" y1="59.69" x2="19.05" y2="59.81" width="0.6096" layer="16"/>
+<wire x1="16.51" y1="67.31" x2="19.05" y2="69.85" width="0.6096" layer="16"/>
+<wire x1="19.05" y1="69.85" x2="48.26" y2="69.85" width="0.6096" layer="16"/>
+<wire x1="48.26" y1="69.85" x2="50.292" y2="67.818" width="0.6096" layer="16"/>
+<wire x1="50.292" y1="67.818" x2="50.292" y2="59.182" width="0.6096" layer="16"/>
+<wire x1="50.292" y1="59.182" x2="48.26" y2="57.15" width="0.6096" layer="16"/>
+<wire x1="48.26" y1="57.15" x2="41.91" y2="57.15" width="0.6096" layer="16"/>
 </signal>
 <signal name="3.3V">
@@
 <wire x1="31.75" y1="43.31" x2="38.224" y2="43.31" width="0.6096" layer="16"/>
 <wire x1="38.224" y1="43.31" x2="38.608" y2="42.926" width="0.6096" layer="16"/>
-<wire x1="41.91" y1="43.18" x2="41.91" y2="50.8" width="0" layer="19" extent="1-1"/>
+<contactref element="R4" pad="2"/>
+<contactref element="R3" pad="2"/>
+<wire x1="38.42" y1="68.26" x2="38.1" y2="68.58" width="0.6096" layer="16"/>
+<wire x1="38.1" y1="68.58" x2="34.29" y2="68.58" width="0.6096" layer="16"/>
+<wire x1="34.29" y1="68.58" x2="33.02" y2="67.31" width="0.6096" layer="16"/>
+<wire x1="33.02" y1="67.31" x2="33.02" y2="66.36" width="0.6096" layer="16"/>
+<wire x1="33.02" y1="66.36" x2="33.34" y2="66.04" width="0.6096" layer="16"/>
+<wire x1="41.91" y1="43.18" x2="44.45" y2="43.18" width="0.6096" layer="16"/>
+<wire x1="44.45" y1="43.18" x2="46.99" y2="45.72" width="0.6096" layer="16"/>
+<wire x1="46.99" y1="45.72" x2="46.99" y2="49.53" width="0.6096" layer="16"/>
+<wire x1="46.99" y1="49.53" x2="45.72" y2="50.8" width="0.6096" layer="16"/>
+<wire x1="45.72" y1="50.8" x2="41.91" y2="50.8" width="0.6096" layer="16"/>
+<wire x1="38.42" y1="66.04" x2="38.42" y2="67.63" width="0.6096" layer="16"/>
+<wire x1="38.42" y1="67.63" x2="39.37" y2="68.58" width="0.6096" layer="16"/>
+<wire x1="44.45" y1="68.58" x2="48.26" y2="64.77" width="0.6096" layer="16"/>
+<wire x1="48.26" y1="60.96" x2="46.482" y2="59.182" width="0.6096" layer="16"/>
+<wire x1="46.482" y1="59.182" x2="39.116" y2="59.182" width="0.6096" layer="16"/>
+<wire x1="39.116" y1="59.182" x2="37.338" y2="57.404" width="0.6096" layer="16"/>
+<wire x1="37.338" y1="57.404" x2="37.338" y2="52.578" width="0.6096" layer="16"/>
+<wire x1="37.338" y1="52.578" x2="39.116" y2="50.8" width="0.6096" layer="16"/>
+<wire x1="39.116" y1="50.8" x2="41.91" y2="50.8" width="0.6096" layer="16"/>
+<wire x1="48.26" y1="60.96" x2="48.26" y2="64.77" width="0.6096" layer="16"/>
+<wire x1="39.37" y1="68.58" x2="44.45" y2="68.58" width="0.6096" layer="16"/>
+<wire x1="38.42" y1="67.63" x2="38.42" y2="68.26" width="0.6096" layer="16"/>
 </signal>
 <signal name="N$2">
@@
 <wire x1="31.75" y1="59.81" x2="31.87" y2="59.69" width="0.6096" layer="16"/>
 <wire x1="31.87" y1="59.69" x2="34.29" y2="59.69" width="0.6096" layer="16"/>
-<wire x1="34.29" y1="59.69" x2="38.1" y2="63.5" width="0.6096" layer="16"/>
+<wire x1="34.29" y1="59.69" x2="36.83" y2="62.23" width="0.6096" layer="16"/>
+<wire x1="36.83" y1="62.23" x2="38.1" y2="63.5" width="0.6096" layer="16"/>
 <wire x1="38.1" y1="63.5" x2="41.91" y2="63.5" width="0.6096" layer="16"/>
+<contactref element="R3" pad="1"/>
+<wire x1="35.24" y1="66.04" x2="35.24" y2="63.82" width="0.6096" layer="16"/>
+<wire x1="35.24" y1="63.82" x2="36.83" y2="62.23" width="0.6096" layer="16"/>
 </signal>
 <signal name="N$8">
@@
 <wire x1="38.1" y1="60.96" x2="35.45" y2="58.31" width="0.6096" layer="16"/>
 <wire x1="35.45" y1="58.31" x2="31.75" y2="58.31" width="0.6096" layer="16"/>
+<contactref element="R4" pad="1"/>
+<wire x1="40.32" y1="66.04" x2="44.45" y2="66.04" width="0.6096" layer="16"/>
+<wire x1="44.45" y1="66.04" x2="45.72" y2="64.77" width="0.6096" layer="16"/>
+<wire x1="45.72" y1="64.77" x2="45.72" y2="62.23" width="0.6096" layer="16"/>
+<wire x1="45.72" y1="62.23" x2="44.45" y2="60.96" width="0.6096" layer="16"/>
+<wire x1="44.45" y1="60.96" x2="41.91" y2="60.96" width="0.6096" layer="16"/>
 </signal>
 <signal name="N$6">
